File: Smartwatch_PCB/Smart watch.kicad_pcb (KiCad board)
At the start: 2 copper layers, 51 parts, among them M1 MS5607, P1 USB_PWR, P2 JTAG_CONN, P3 BATT_CONN, SW1 SW_PUSH, Y2 8MHZ

Commit message: Final version...I hope
Parts:
- added SW2: SW_PUSH, Buttons_Switches_ThroughHole:SW_PUSH_SMALL, F.Cu at (140.4, 112.0)
- moved C19 6.82 mm to (140.6, 101.8)
- moved LS1 6.82 mm to (139.5, 95.7)
- moved C20 6.82 mm to (140.5, 89.6)
- moved C21 6.82 mm to (136.5, 95.6)
Connections:
- BT1 pad 1: Net-(BT1-Pad1) -> (no net)
- BT1 pad 10: Net-(BT1-Pad10) -> (no net)
- BT1 pad 13: Net-(BT1-Pad13) -> (no net)
- BT1 pad 14: Net-(BT1-Pad14) -> (no net)
- BT1 pad 15: Net-(BT1-Pad15) -> (no net)
- BT1 pad 16: Net-(BT1-Pad16) -> (no net)
- BT1 pad 3: Net-(BT1-Pad3) -> (no net)
- BT1 pad 5: Net-(BT1-Pad5) -> (no net)
- BT1 pad 6: Net-(BT1-Pad6) -> (no net)
- BT1 pad 7: Net-(BT1-Pad7) -> (no net)
- BT1 pad 8: Net-(BT1-Pad8) -> (no net)
- M1 pad 6: Net-(M1-Pad6) -> (no net)
- MAX1 pad 4: Net-(MAX1-Pad4) -> (no net)
- P1 pad 2: Net-(P1-Pad2) -> (no net)
- P1 pad 3: Net-(P1-Pad3) -> (no net)
- P1 pad 5: Net-(P1-Pad5) -> (no net)
- S1 pad 3: Net-(S1-Pad3) -> (no net)
- S1 pad 4: Net-(S1-Pad4) -> (no net)
- UCL1 pad 10: Net-(UCL1-Pad10) -> (no net)
- UCL1 pad 11: Net-(UCL1-Pad11) -> (no net)
- UCL1 pad 14: Net-(UCL1-Pad14) -> (no net)
- UCL1 pad 15: Net-(UCL1-Pad15) -> (no net)
- UCL1 pad 2: Net-(UCL1-Pad2) -> (no net)
- UCL1 pad 25: Net-(UCL1-Pad25) -> (no net)
- UCL1 pad 26: Net-(UCL1-Pad26) -> (no net)
- UCL1 pad 27: Net-(UCL1-Pad27) -> (no net)
- UCL1 pad 29: Net-(UCL1-Pad29) -> (no net)
- UCL1 pad 30: Net-(UCL1-Pad30) -> (no net)
- UCL1 pad 33: Net-(UCL1-Pad33) -> (no net)
- UCL1 pad 34: Net-(UCL1-Pad34) -> (no net)
- UCL1 pad 35: Net-(UCL1-Pad35) -> (no net)
- UCL1 pad 36: Net-(UCL1-Pad36) -> (no net)
- UCL1 pad 37: Net-(UCL1-Pad37) -> (no net)
- UCL1 pad 38: Net-(UCL1-Pad38) -> (no net)
- UCL1 pad 39: Net-(UCL1-Pad39) -> (no net)
- UCL1 pad 40: Net-(UCL1-Pad40) -> (no net)
- UCL1 pad 41: Net-(UCL1-Pad41) -> (no net)
- UCL1 pad 44: Net-(UCL1-Pad44) -> (no net)
- UCL1 pad 45: Net-(UCL1-Pad45) -> (no net)
- UCL1 pad 51: Net-(UCL1-Pad51) -> (no net)
- UCL1 pad 52: Net-(UCL1-Pad52) -> (no net)
- UCL1 pad 53: Net-(UCL1-Pad53) -> (no net)
- UCL1 pad 54: Net-(UCL1-Pad54) -> (no net)
- UCL1 pad 57: Net-(UCL1-Pad57) -> (no net)
- UCL1 pad 61: Net-(UCL1-Pad61) -> (no net)
- UCL1 pad 62: Net-(UCL1-Pad62) -> (no net)
- UCL1 pad 9: Net-(UCL1-Pad9) -> (no net)
Routing:
- net Net-(SW2-Pad2): track 0.00 -> 32.6 mm, vias 0 -> 2
- net GND: track 370.8 -> 384.0 mm
- net /3.3V: track 223.9 -> 228.7 mm
- net /LCD_ON_OFF: track 31.3 -> 33.2 mm
- net /SPI1_SCK: track 26.3 -> 24.5 mm
- net /SPI1_MOSI: track 27.6 -> 25.8 mm
- net /SPI_CS: track 20.1 -> 21.5 mm
- net /TDI: track 24.8 -> 23.4 mm
- net /USART_RX: track 31.4 -> 32.4 mm
- net /TDO/SWO: track 32.3 -> 33.2 mm
- net /RESET: track 146.2 -> 146.8 mm
- net /EXTCLCK: track 23.8 -> 24.5 mm
- net /USART_TX: track 29.1 -> 28.5 mm
Other:
- board outline added: 69.3 x 63.8 mm
- net class Default: clearance 0.2 -> 0.199
- rule trace_clearance: 0.2 -> 0.199
