File: Smartwatch_PCB/Smart watch.sch (KiCad schematic (older format))
At the start: 47 parts, among them M1 MS5607, P1 USB_PWR, P2 JTAG_CONN, P3 BATT_CONN, SW1 SW_PUSH, Y2 8MHZ

Commit message: Final version...I hope
Parts:
- added SW2: SW_PUSH, Buttons_Switches_ThroughHole:SW_PUSH_SMALL, symbol SW_PUSH
Connections:
- net GND: now also SW2.1
- net at UCL1.17 (PA3): now also SW2.2
- no-connect marks 48 -> 47
Changed lines of the file:
@@
 NoConn ~ 8400 10750
 NoConn ~ 8400 10950
-NoConn ~ 9200 12750
 NoConn ~ 10800 12750
 NoConn ~ 11000 12750
@@
 	8100 11350 8100 11400
 Connection ~ 8100 11350
+$Comp
+L SW_PUSH SW2
+U 1 1 56731C68
+P 8500 12900
+F 0 "SW2" H 8650 13010 50  0000 C CNN
+F 1 "SW_PUSH" H 8500 12820 50  0000 C CNN
+F 2 "Buttons_Switches_ThroughHole:SW_PUSH_SMALL" H 8500 12900 50  0001 C CNN
+F 3 "" H 8500 12900 50  0000 C CNN
+	1    8500 12900
+	1    0    0    -1
+$EndComp
+Wire Wire Line
+	9200 12750 9200 12900
+Wire Wire Line
+	9200 12900 8800 12900
+$Comp
+L GND #PWR037
+U 1 1 56731E60
+P 7950 13050
+F 0 "#PWR037" H 7950 12800 50  0001 C CNN
+F 1 "GND" H 7950 12900 50  0000 C CNN
+F 2 "" H 7950 13050 50  0000 C CNN
+F 3 "" H 7950 13050 50  0000 C CNN
+	1    7950 13050
+	1    0    0    -1
+$EndComp
+Wire Wire Line
+	8200 12900 7950 12900
+Wire Wire Line
+	7950 12900 7950 13050
 $EndSCHEMATC
